File: hardware/Aeroq Hardware v3.kicad_pcb (KiCad board)
At the start: 2 copper layers, 45 x 45 mm, 59 parts, among them J1 2x4 male header 2.54 mm, J2 USB4120-03-C, J3 SM06B-GHS-TB, J4 FH12A-24S-0.5SH(55), Q1 Si1308EDL, U1 TLV76133DCY, U2 ESP32-C3-MINI-1-N4, U3 SCD40-D-R2

Commit message: updates
Parts:
- removed D2: SMAJ5.0CA, Diode_SMD:D_SMA
- removed D3, D4: ESD321DYAR, Package_TO_SOT_SMD:SOT-523
- added U4: USBLC6-2SC6, Package_TO_SOT_SMD:SOT-23-6, F.Cu at (113.7, 107.0)
- U3: footprint Sensor:Sensirion_SCD4x-1EP_10.1x10.1mm_P1.25mm_EP4.8x4.8mm -> 2s_misc:Sensirion_SCD4x-1EP_10.1x10.1mm_P1.25mm_EP4.8x4.8mm
- moved FID3 6.86 mm to (88.7, 82.1)
- moved R12 2.42 mm to (110.0, 113.2), turned to -90 degrees
- moved FID2 0.46 mm to (101.0, 117.5)
Routing:
- net VBUS: track 41.9 -> 35.7 mm, vias 6 -> 2
- net /USB-C/D-: track 39.1 -> 41.2 mm, vias 2 -> 4
- net /USB-C/D+: track 40.7 -> 39.1 mm, vias 2 -> 0
- net Net-(J2-CC1): track 6.94 -> 8.17 mm
- net /Display/RESE: track 16.8 -> 15.8 mm
- net +3.3V: track 45.0 -> 44.1 mm
Other:
- board text added: "luftaq v1.0"
