File: hardware/microcontroller.kicad_sch (KiCad schematic)
At the start: 14 parts, among them J1 2x4 male header 2.54 mm, U2 ESP32-C3-MINI-1-N4

Commit message: updates
Connections:
- no-connect marks 1 -> 0
Changed lines of the file:
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@@
 		(color 0 0 0 0)
-	)
-	(no_connect
-		(at 226.06 157.48)
 	)
 	(wire
