File: hardware/sensors.kicad_sch (KiCad schematic)
At the start: 6 parts, among them J3 SM06B-GHS-TB, U3 SCD40-D-R2

Commit message: updates
Parts:
- U3: footprint Sensor:Sensirion_SCD4x-1EP_10.1x10.1mm_P1.25mm_EP4.8x4.8mm -> 2s_misc:Sensirion_SCD4x-1EP_10.1x10.1mm_P1.25mm_EP4.8x4.8mm
Changed lines of the file:
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@@
 			)
 		)
-		(property "Footprint" "Sensor:Sensirion_SCD4x-1EP_10.1x10.1mm_P1.25mm_EP4.8x4.8mm"
+		(property "Footprint" "2s_misc:Sensirion_SCD4x-1EP_10.1x10.1mm_P1.25mm_EP4.8x4.8mm"
 			(at 149.86 113.03 0)
 			(effects
