File: hardware/usb-c.kicad_sch (KiCad schematic)
At the start: 7 parts, among them J2 USB4120-03-C

Commit message: updates
Parts:
- removed D2: SMAJ5.0CA, Diode_SMD:D_SMA, symbol 2s_diodes:SMAJ5.0CA
- removed D3, D4: ESD321DYAR, Package_TO_SOT_SMD:SOT-523, symbol 2s_diodes:ESD321DYAR
- added U4: USBLC6-2SC6, Package_TO_SOT_SMD:SOT-23-6, symbol 2s_diodes:USBLC6-2SC6
Connections:
- net D+: now also U4.1 (I/O1)
- net D-: now also U4.4 (I/O2)
- net GND: now also U4.2 (GND)
- net VBUS: now also U4.5 (VBUS)
- no-connect marks 6 -> 8
Other:
- moved on the sheet: R13

Commit message: fix whitespace in MPN
Parts:
- U4: MPN (none) -> USBLC6-2SC6
Changed lines of the file:
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@@
+			)
+		)
+		(property "MPN" "USBLC6-2SC6"
+			(at 262.89 153.67 0)
+			(effects
+				(font
+					(size 1.27 1.27)
+				)
+				(hide yes)
 			)
 		)
